File: camera_routing.kicad_pcb (KiCad board)
At the start: 6 copper layers, 4 parts, among them U1 111, U28 NC

Commit message: added ground fill
Routing:
- added copper zone on F.Cu, net GND
Other:
- board outline added: 34.3 x 34.3 mm
